Commit message: update xacro - bodyshape

File: neurobot_virtual/src/nebot_description/urdf/nebot.xacro (robot description, xacro)
@@ -31,5 +31,5 @@
       <origin xyz="0.05 0 0.05" rpy=" 0 0 0"/>
       <geometry>
-        <box size="0.3 0.16 0.005"/> <!--less to improve sensors-->
+        <box size="0.24 0.16 0.005"/> <!--less to improve sensors-->
       </geometry>
     </collision>
@@ -354,5 +354,5 @@
   <joint name="sonar_front_joint" type="fixed">
     <axis xyz="0 1 0" />
-    <origin rpy="0 0 0" xyz="0.18 0 0.06" />
+    <origin rpy="0 0 0" xyz="0.19 0 0.06" />
     <parent link="chassis"/>
     <child link="base_sonar_front"/>
@@ -379,5 +379,5 @@
   <joint name="sonar_right_joint" type="fixed">
     <axis xyz="0 1 0" />
-    <origin rpy="0 0 0.523" xyz="0.175 0.06 0.06" />
+    <origin rpy="0 0 0.523" xyz="0.185 0.06 0.06" />
     <parent link="chassis"/>
     <child link="base_sonar_right"/>
@@ -404,5 +404,5 @@
   <joint name="sonar_left_joint" type="fixed">
     <axis xyz="0 1 0" />
-    <origin rpy="0 0 -0.523" xyz="0.175 -0.06 0.06" />
+    <origin rpy="0 0 -0.523" xyz="0.185 -0.06 0.06" />
     <parent link="chassis"/>
     <child link="base_sonar_left"/>
@@ -429,5 +429,5 @@
   <joint name="sonar_back_joint" type="fixed">
     <axis xyz="0 1 0" />
-    <origin rpy="0 0 3.14" xyz="-0.2 0 0.05" />
+    <origin rpy="0 0 3.14" xyz="-0.21 0 0.05" />
     <parent link="chassis"/>
     <child link="back_sonar_forward"/>
@@ -449,5 +449,5 @@
   <joint name="sonar_back2_joint" type="fixed">
     <axis xyz="0 1 0" />
-    <origin rpy="0 0 2.617" xyz="-0.19 0.06 0.05" />
+    <origin rpy="0 0 2.617" xyz="-0.20 0.06 0.05" />
     <parent link="chassis"/>
     <child link="back_sonar_left"/>
@@ -469,5 +469,5 @@
   <joint name="sonar_back3_joint" type="fixed">
     <axis xyz="0 1 0" />
-    <origin rpy="0 0 3.663" xyz="-0.19 -0.06 0.05" />
+    <origin rpy="0 0 3.663" xyz="-0.20 -0.06 0.05" />
     <parent link="chassis"/>
     <child link="back_sonar_right"/>
